File: hardware/ToneLock/MCU.sch (EAGLE design)
At the start: 46 parts, among them Q1 IRLML6346, U1 LD1117S33TR, U2 MP45DT02, U3 LIS3DSHTR, X3 MINI-USB-32005-201

Commit message: Routed, polygon poured, ready in theory
Parts:
- added TP1: TPB1,27, testpad:TPB1,27
- C15, C16: device resistor:C-EUC0603 -> resistor:C-EUC0805
Connections:
- net MIC_PDM: now also TP1.TP
Other:
- moved on the sheet: U1
Changed lines of the file:
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@@
 <part name="SV2" library="con-lstb" library_urn="urn:adsk.eagle:library:162" deviceset="MA05-1" device="" package3d_urn="urn:adsk.eagle:package:8332/1"/>
 <part name="GND13" library="supply1" library_urn="urn:adsk.eagle:library:371" deviceset="GND" device=""/>
-<part name="C15" library="resistor" library_urn="urn:adsk.eagle:library:348" deviceset="C-EU" device="C0603" package3d_urn="urn:adsk.eagle:package:23616/2" value="10uF"/>
-<part name="C16" library="resistor" library_urn="urn:adsk.eagle:library:348" deviceset="C-EU" device="C0603" package3d_urn="urn:adsk.eagle:package:23616/2" value="10uF"/>
+<part name="C15" library="resistor" library_urn="urn:adsk.eagle:library:348" deviceset="C-EU" device="C0805" package3d_urn="urn:adsk.eagle:package:23617/2" value="10uF"/>
+<part name="C16" library="resistor" library_urn="urn:adsk.eagle:library:348" deviceset="C-EU" device="C0805" package3d_urn="urn:adsk.eagle:package:23617/2" value="10uF"/>
 <part name="DBG_LED1" library="led" library_urn="urn:adsk.eagle:library:259" deviceset="LED" device="CHIP-LED0603" package3d_urn="urn:adsk.eagle:package:15819/3"/>
 <part name="GND15" library="supply1" library_urn="urn:adsk.eagle:library:371" deviceset="GND" device=""/>
@@
 <part name="P+5" library="supply1" library_urn="urn:adsk.eagle:library:371" deviceset="+12V" device=""/>
 <part name="C17" library="resistor" library_urn="urn:adsk.eagle:library:348" deviceset="C-EU" device="C0603" package3d_urn="urn:adsk.eagle:package:23616/2" value="100nF"/>
+<part name="TP1" library="testpad" library_urn="urn:adsk.eagle:library:385" deviceset="TP" device="B1,27" package3d_urn="urn:adsk.eagle:package:27944/1" value="TPB1,27"/>
 </parts>
 <sheets>
@@
 </instance>
 <instance part="C17" gate="G$1" x="-68.58" y="134.62"/>
+<instance part="TP1" gate="G$1" x="144.78" y="96.52" rot="R270"/>
 </instances>
 <busses>
@@
 <label x="121.92" y="86.36" size="1.27" layer="95" xref="yes"/>
 </segment>
-</net>
+<segment>
+<pinref part="TP1" gate="G$1" pin="TP"/>
+<wire x1="142.24" y1="96.52" x2="139.7" y2="96.52" width="0.1524" layer="91"/>
+<label x="139.7" y="96.52" size="1.778" layer="95" rot="R180" xref="yes"/>
+</segment>
+</net>

Commit message: Ready for polygon
Connections:
- removed net MEMS_CS: U$1.PE3, U3.CS
- new net MEMS_NCS: U$1.PE8, U3.CS
- net MEMS_INT1: now also U$1.PE10; no longer U$1.PE0
- net MEMS_INT2: now also U$1.PE11; no longer U$1.PE1
Changed lines of the file:
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@@
-</segment>
-</net>
-<net name="MEMS_CS" class="0">
-<segment>
-<wire x1="93.98" y1="147.32" x2="91.44" y2="147.32" width="0.1524" layer="91"/>
-<label x="91.44" y="147.32" size="1.27" layer="95" rot="R180" xref="yes"/>
-<pinref part="U3" gate="G$1" pin="CS"/>
-</segment>
-<segment>
-<wire x1="50.8" y1="43.18" x2="53.34" y2="43.18" width="0.1524" layer="91"/>
-<label x="53.34" y="43.18" size="1.27" layer="95" xref="yes"/>
-<pinref part="U$1" gate="G$1" pin="PE3"/>
 </segment>
 </net>
 <net name="MEMS_INT1" class="0">
-<segment>
-<wire x1="50.8" y1="50.8" x2="53.34" y2="50.8" width="0.1524" layer="91"/>
-<label x="53.34" y="50.8" size="1.27" layer="95" xref="yes"/>
-<pinref part="U$1" gate="G$1" pin="PE0"/>
-</segment>
 <segment>
 <pinref part="U3" gate="G$1" pin="INT1"/>
@@
 <label x="91.44" y="139.7" size="1.27" layer="95" rot="R180" xref="yes"/>
 </segment>
+<segment>
+<pinref part="U$1" gate="G$1" pin="PE10"/>
+<wire x1="50.8" y1="25.4" x2="53.34" y2="25.4" width="0.1524" layer="91"/>
+<label x="53.34" y="25.4" size="1.27" layer="95" xref="yes"/>
+</segment>
 </net>
 <net name="MEMS_INT2" class="0">
-<segment>
-<wire x1="50.8" y1="48.26" x2="53.34" y2="48.26" width="0.1524" layer="91"/>
-<label x="53.34" y="48.26" size="1.27" layer="95" xref="yes"/>
-<pinref part="U$1" gate="G$1" pin="PE1"/>
-</segment>
 <segment>
 <pinref part="U3" gate="G$1" pin="INT2"/>
 <wire x1="93.98" y1="137.16" x2="91.44" y2="137.16" width="0.1524" layer="91"/>
 <label x="91.44" y="137.16" size="1.27" layer="95" rot="R180" xref="yes"/>
+</segment>
+<segment>
+<pinref part="U$1" gate="G$1" pin="PE11"/>
+<wire x1="50.8" y1="22.86" x2="53.34" y2="22.86" width="0.1524" layer="91"/>
+<label x="53.34" y="22.86" size="1.27" layer="95" xref="yes"/>
 </segment>
 </net>
@@
 </segment>
 </net>
+<net name="MEMS_NCS" class="0">
+<segment>
+<wire x1="93.98" y1="147.32" x2="91.44" y2="147.32" width="0.1524" layer="91"/>
+<label x="91.44" y="147.32" size="1.27" layer="95" rot="R180" xref="yes"/>
+<pinref part="U3" gate="G$1" pin="CS"/>
+</segment>
+<segment>
+<pinref part="U$1" gate="G$1" pin="PE8"/>
+<wire x1="50.8" y1="30.48" x2="53.34" y2="30.48" width="0.1524" layer="91"/>
+<label x="53.34" y="30.48" size="1.27" layer="95" xref="yes"/>
+</segment>
+</net>

Commit message: Hardware ready to generate gerber
Parts:
- added TP2, TP3: TPB2,54, testpad:TPB2,54
- TP1: value TPB1,27 -> TPB2,54; device testpad:TPB1,27 -> testpad:TPB2,54
Connections:
- net MEMS_SCK: now also TP3.TP
- net MIC_CLK: now also TP2.TP
Other:
- moved on the sheet: TP1
Changed lines of the file:
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@@
 <part name="P+5" library="supply1" library_urn="urn:adsk.eagle:library:371" deviceset="+12V" device=""/>
 <part name="C17" library="resistor" library_urn="urn:adsk.eagle:library:348" deviceset="C-EU" device="C0603" package3d_urn="urn:adsk.eagle:package:23616/2" value="100nF"/>
-<part name="TP1" library="testpad" library_urn="urn:adsk.eagle:library:385" deviceset="TP" device="B1,27" package3d_urn="urn:adsk.eagle:package:27944/1" value="TPB1,27"/>
+<part name="TP1" library="testpad" library_urn="urn:adsk.eagle:library:385" deviceset="TP" device="B2,54" package3d_urn="urn:adsk.eagle:package:27948/1" value="TPB2,54"/>
+<part name="TP2" library="testpad" library_urn="urn:adsk.eagle:library:385" deviceset="TP" device="B2,54" package3d_urn="urn:adsk.eagle:package:27948/1"/>
+<part name="TP3" library="testpad" library_urn="urn:adsk.eagle:library:385" deviceset="TP" device="B2,54" package3d_urn="urn:adsk.eagle:package:27948/1"/>
 </parts>
 <sheets>
@@
 </instance>
 <instance part="C17" gate="G$1" x="-68.58" y="134.62"/>
-<instance part="TP1" gate="G$1" x="144.78" y="96.52" rot="R270"/>
+<instance part="TP1" gate="G$1" x="149.86" y="104.14" rot="R270"/>
+<instance part="TP2" gate="G$1" x="149.86" y="99.06" rot="R270"/>
+<instance part="TP3" gate="G$1" x="149.86" y="93.98" rot="R270"/>
 </instances>
 <busses>
@@
 <label x="91.44" y="132.08" size="1.27" layer="95" rot="R180" xref="yes"/>
 </segment>
+<segment>
+<pinref part="TP3" gate="G$1" pin="TP"/>
+<wire x1="147.32" y1="93.98" x2="144.78" y2="93.98" width="0.1524" layer="91"/>
+<label x="144.78" y="93.98" size="1.27" layer="95" rot="R180" xref="yes"/>
+</segment>
 </net>
 <net name="MEMS_MOSI" class="0">
@@
 <segment>
 <pinref part="TP1" gate="G$1" pin="TP"/>
-<wire x1="142.24" y1="96.52" x2="139.7" y2="96.52" width="0.1524" layer="91"/>
-<label x="139.7" y="96.52" size="1.778" layer="95" rot="R180" xref="yes"/>
+<wire x1="147.32" y1="104.14" x2="144.78" y2="104.14" width="0.1524" layer="91"/>
+<label x="144.78" y="104.14" size="1.27" layer="95" rot="R180" xref="yes"/>
 </segment>
 </net>
@@
 <label x="121.92" y="83.82" size="1.27" layer="95" xref="yes"/>
 </segment>
-</net>
+<segment>
+<pinref part="TP2" gate="G$1" pin="TP"/>
+<wire x1="147.32" y1="99.06" x2="144.78" y2="99.06" width="0.1524" layer="91"/>
+<label x="144.78" y="99.06" size="1.27" layer="95" rot="R180" xref="yes"/>
+</segment>
+</net>
